File: hardware/switch-connector/switch-box.sch (KiCad schematic (older format))
At the start: 10 parts, among them P1 12V, P2 Relay OFF (NC), P3 Sensing, P4 GND, P5 Relay On enable (NO), P6 Sustain, P7 Trigger, SW1 NC: Off, SW2 NO: On, SW3 NC: E-Stop

Commit message: o Update board with new connectors.
Parts:
- removed P4: GND, Pin_Headers:Pin_Header_Straight_1x01, symbol CONN_01X01
- removed P6: Sustain, Pin_Headers:Pin_Header_Straight_1x01, symbol CONN_01X01
- removed P7: Trigger, Pin_Headers:Pin_Header_Straight_1x01, symbol CONN_01X01
- added P4: SwitchConnector, Pin_Headers:Pin_Header_Straight_1x05, symbol CONN_01X05
- added P6: HV-RelayConnector, Pin_Headers:Pin_Header_Straight_1x04, symbol CONN_01X03
- P2: value Relay OFF (NC) -> Force OFF (NC)
- P5: value Relay On enable (NO) -> Enable ON (NO)
- SW1, SW2, SW3: footprint Pin_Headers:Pin_Header_Straight_1x02 -> (none)
Connections:
- wire segments 25 -> 37
Changed lines of the file:
@@
 F 0 "SW1" H 2800 2710 50  0000 C CNN
 F 1 "NC: Off" H 2650 2520 50  0000 C CNN
-F 2 "Pin_Headers:Pin_Header_Straight_1x02" H 2650 2600 50  0001 C CNN
+F 2 "" H 2650 2600 50  0001 C CNN
 F 3 "" H 2650 2600 50  0000 C CNN
 	1    2650 2600
@@
 	-1   0    0    1
 $EndComp
-Wire Notes Line
-	3650 3400 3650 3550
-Wire Notes Line
-	3600 3550 3700 3550
-Wire Notes Line
-	3600 3550 3600 3700
-Wire Notes Line
-	3600 3700 3700 3700
-Wire Notes Line
-	3700 3700 3700 3550
-Wire Notes Line
-	3650 3700 3650 3750
-Wire Notes Line
-	3650 3750 3950 3750
-Wire Notes Line
-	3900 3750 3900 3700
-Wire Wire Line
-	1350 3000 3700 3000
-Wire Wire Line
-	3250 2900 3800 2900
-Wire Wire Line
-	3800 2900 3800 3000
-Wire Wire Line
-	4050 2950 3900 2950
-Wire Wire Line
-	3900 2950 3900 3000
-Wire Notes Line
-	3800 3400 3800 3550
-Wire Notes Line
-	3950 3750 3950 3400
 $Comp
 L SW_PUSH SW2
@@
 F 0 "SW2" H 3800 2710 50  0000 C CNN
 F 1 "NO: On" H 3650 2520 50  0000 C CNN
-F 2 "Pin_Headers:Pin_Header_Straight_1x02" H 3650 2600 50  0001 C CNN
+F 2 "" H 3650 2600 50  0001 C CNN
 F 3 "" H 3650 2600 50  0000 C CNN
 	1    3650 2600
 	1    0    0    -1
 $EndComp
-Wire Wire Line
-	3100 2600 3350 2600
-Wire Wire Line
-	3250 2400 3250 2900
-Connection ~ 3250 2600
 $Comp
 L CONN_01X02 P5
@@
 P 4000 2100
 F 0 "P5" H 4000 2250 50  0000 C CNN
-F 1 "Relay On enable (NO)" V 4100 1800 50  0000 C CNN
+F 1 "Enable ON (NO)" V 4100 2100 50  0000 C CNN
 F 2 "Pin_Headers:Pin_Header_Straight_1x02" H 4000 2100 50  0001 C CNN
 F 3 "" H 4000 2100 50  0000 C CNN
@@
 	0    -1   -1   0
 $EndComp
-Wire Wire Line
-	3950 2300 3950 2600
-Wire Wire Line
-	4050 2300 4050 2950
 $Comp
 L CONN_01X02 P2
@@
 P 3050 2100
 F 0 "P2" H 3050 2250 50  0000 C CNN
-F 1 "Relay OFF (NC)" V 3150 2250 50  0000 C CNN
+F 1 "Force OFF (NC)" V 3150 2250 50  0000 C CNN
 F 2 "Pin_Headers:Pin_Header_Straight_1x02" H 3050 2100 50  0001 C CNN
 F 3 "" H 3050 2100 50  0000 C CNN
@@
 	0    -1   -1   0
 $EndComp
-Wire Wire Line
-	3000 2300 3000 2600
-Wire Wire Line
-	3000 2600 2950 2600
-Wire Wire Line
-	3100 2300 3100 2600
-Wire Wire Line
-	3400 2400 3250 2400
-Wire Wire Line
-	3600 2300 4050 2300
-Connection ~ 4050 2300
-Wire Wire Line
-	3500 1900 3500 2400
-Wire Wire Line
-	3500 2400 3950 2400
-Connection ~ 3950 2400
 $Comp
 L SW_PUSH SW3
@@
 F 0 "SW3" H 2000 2710 50  0000 C CNN
 F 1 "NC: E-Stop" H 1850 2520 50  0000 C CNN
-F 2 "Pin_Headers:Pin_Header_Straight_1x02" H 1850 2600 50  0001 C CNN
+F 2 "" H 1850 2600 50  0001 C CNN
 F 3 "" H 1850 2600 50  0000 C CNN
 	1    1850 2600
@@
 	0    -1   -1   0
 $EndComp
-Wire Wire Line
-	2150 2600 2350 2600
-Wire Wire Line
-	3300 2300 2300 2300
-Wire Wire Line
-	2300 2300 2300 2600
-Connection ~ 2300 2600
-Wire Wire Line
-	1550 2600 1350 2600
-Wire Wire Line
-	1350 2600 1350 2700
-Wire Wire Line
-	1350 2800 1350 3000
-$Comp
-L CONN_01X01 P4
-U 1 1 57D0BFC6
-P 3700 3200
-F 0 "P4" H 3700 3300 50  0000 C CNN
-F 1 "GND" V 3850 3050 50  0000 C CNN
-F 2 "Pin_Headers:Pin_Header_Straight_1x01" H 3700 3200 50  0001 C CNN
-F 3 "" H 3700 3200 50  0000 C CNN
-	1    3700 3200
-	0    1    1    0
-$EndComp
-$Comp
-L CONN_01X01 P6
-U 1 1 57D0BFFC
-P 3800 3200
-F 0 "P6" H 3800 3300 50  0000 C CNN
-F 1 "Sustain" V 3950 3200 50  0000 C CNN
-F 2 "Pin_Headers:Pin_Header_Straight_1x01" H 3800 3200 50  0001 C CNN
-F 3 "" H 3800 3200 50  0000 C CNN
-	1    3800 3200
-	0    1    1    0
-$EndComp
-$Comp
-L CONN_01X01 P7
-U 1 1 57D0C02A
-P 3900 3200
-F 0 "P7" H 3900 3300 50  0000 C CNN
-F 1 "Trigger" V 4050 3400 50  0000 C CNN
-F 2 "Pin_Headers:Pin_Header_Straight_1x01" H 3900 3200 50  0001 C CNN
-F 3 "" H 3900 3200 50  0000 C CNN
-	1    3900 3200
-	0    1    1    0
-$EndComp
-Text HLabel 4050 2900 2    60   Output ~ 0
+Text HLabel 3900 3450 3    60   Output ~ 0
 Trigger
-Text Notes 3750 3650 0    60   ~ 0
+Text Notes 3750 4200 0    60   ~ 0
 NO
-Text Notes 4050 3700 0    60   ~ 0
+Text Notes 4050 4250 0    60   ~ 0
 2 more switches\nfor HV switching
-Text HLabel 3250 2800 2    60   Output ~ 0
+Text HLabel 3800 3450 3    60   Output ~ 0
 Sustain
 $Comp
-L GND #PWR?
+L GND #PWR01
 U 1 1 58AB6D12
 P 1450 3000
-F 0 "#PWR?" H 1450 2750 50  0001 C CNN
+F 0 "#PWR01" H 1450 2750 50  0001 C CNN
 F 1 "GND" H 1455 2827 50  0000 C CNN
 F 2 "" H 1450 3000 50  0000 C CNN
@@
 	1    0    0    -1
 $EndComp
-Text HLabel 3350 3000 3    60   Output ~ 0
+Text HLabel 3700 3450 3    60   Output ~ 0
 CoilGnd
 $Comp
-L +12V #PWR?
+L +12V #PWR02
 U 1 1 58AB7391
 P 1450 2600
-F 0 "#PWR?" H 1450 2450 50  0001 C CNN
+F 0 "#PWR02" H 1450 2450 50  0001 C CNN
 F 1 "+12V" H 1465 2773 50  0000 C CNN
 F 2 "" H 1450 2600 50  0000 C CNN
@@
 	1    0    0    -1
 $EndComp
-Connection ~ 1450 3000
-Connection ~ 1450 2600
 Text HLabel 3300 1900 1    60   Output ~ 0
 Sense-E-Stop
@@
 Text HLabel 3600 1900 1    60   Output ~ 0
 Sense-Powered
+Wire Notes Line
+	3650 3950 3650 4100
+Wire Notes Line
+	3600 4100 3700 4100
+Wire Notes Line
+	3600 4100 3600 4250
+Wire Notes Line
+	3600 4250 3700 4250
+Wire Notes Line
+	3700 4250 3700 4100
+Wire Notes Line
+	3650 4250 3650 4300
+Wire Notes Line
+	3650 4300 3950 4300
+Wire Notes Line
+	3900 4300 3900 4250
+Wire Wire Line
+	1350 3000 3700 3000
+Wire Wire Line
+	3800 2850 3800 3450
+Wire Wire Line
+	4050 2950 3900 2950
+Wire Wire Line
+	3900 2950 3900 3450
+Wire Notes Line
+	3800 3950 3800 4100
+Wire Notes Line
+	3950 4300 3950 3950
+Wire Wire Line
+	3100 2600 3350 2600
+Connection ~ 3250 2600
+Wire Wire Line
+	3950 2300 3950 2900
+Wire Wire Line
+	4050 2300 4050 2950
+Wire Wire Line
+	3000 2300 3000 2600
+Wire Wire Line
+	3000 2600 2950 2600
+Wire Wire Line
+	3100 2300 3100 2600
+Wire Wire Line
+	3400 2400 3250 2400
+Wire Wire Line
+	3600 2300 4050 2300
+Connection ~ 4050 2300
+Wire Wire Line
+	3500 1900 3500 2400
+Wire Wire Line
+	3500 2400 3950 2400
+Connection ~ 3950 2400
+Wire Wire Line
+	2150 2600 2350 2600
+Wire Wire Line
+	3300 2300 2300 2300
+Wire Wire Line
+	2300 2300 2300 2750
+Connection ~ 2300 2600
+Wire Wire Line
+	1350 2600 1550 2600
+Wire Wire Line
+	1350 2600 1350 2700
+Wire Wire Line
+	1350 2800 1350 3000
+Connection ~ 1450 3000
+Connection ~ 1450 2600
 Connection ~ 3500 2300
 Wire Wire Line
@@
 Wire Wire Line
 	3600 2300 3600 1900
+$Comp
+L CONN_01X05 P4
+U 1 1 58AB6DAC
+P 2350 3400
+F 0 "P4" V 2222 3678 50  0000 L CNN
+F 1 "SwitchConnector" V 2450 3100 50  0000 L CNN
+F 2 "Pin_Headers:Pin_Header_Straight_1x05" H 2350 3400 50  0001 C CNN
+F 3 "" H 2350 3400 50  0000 C CNN
+	1    2350 3400
+	0    -1   1    0
+$EndComp
+Wire Wire Line
+	1550 2900 2150 2900
+Wire Wire Line
+	2150 2900 2150 3200
+Wire Wire Line
+	1550 2600 1550 2900
+Connection ~ 1550 2600
+Wire Wire Line
+	2300 2750 2250 2750
+Wire Wire Line
+	2250 2750 2250 3200
+Wire Wire Line
+	2950 2600 2950 2800
+Wire Wire Line
+	2950 2800 2350 2800
+Wire Wire Line
+	2350 2800 2350 3200
+Connection ~ 2950 2600
+Wire Wire Line
+	2450 3200 2450 2850
+Wire Wire Line
+	2450 2850 3800 2850
+Wire Wire Line
+	3250 2400 3250 2850
+Connection ~ 3250 2850
+Wire Wire Line
+	2550 3200 2550 2900
+Wire Wire Line
+	2550 2900 3950 2900
+Connection ~ 3950 2600
+$Comp
+L CONN_01X03 P6
+U 1 1 58AB7BE4
+P 3800 3400
+F 0 "P6" V 3672 3212 50  0000 R CNN
+F 1 "HV-RelayConnector" V 3763 3212 50  0000 R CNN
+F 2 "Pin_Headers:Pin_Header_Straight_1x04" H 3809 3212 50  0001 R CNN
+F 3 "" H 3800 3400 50  0000 C CNN
+	1    3800 3400
+	0    -1   1    0
+$EndComp
+Wire Wire Line
+	3700 3000 3700 3450
+Connection ~ 3700 3200
+Connection ~ 3800 3200
+Connection ~ 3900 3200
 $EndSCHEMATC

Commit message: o clarifications in schematic
Parts:
- P2: value Force OFF (NC) -> Force off (NC)
- P5: value Enable ON (NO) -> Enable on (NO)
Connections:
- net labels added: Sense-Sustained
- net labels removed: Sense-Powered
Other:
- note added: "[1, 2]: E-Stop; NC\n[2, 3]: Off; NC (NB: 2 is shared)\n[4, 5]: On; NO\n"
- note added: "with RPi\nswitched Relay"
Changed lines of the file:
@@
 LIBS:relays
 LIBS:parts
+LIBS:switches
 LIBS:switch-connector-cache
 EELAYER 25 0
@@
 P 4000 2100
 F 0 "P5" H 4000 2250 50  0000 C CNN
-F 1 "Enable ON (NO)" V 4100 2100 50  0000 C CNN
+F 1 "Enable on (NO)" V 4100 2100 50  0000 C CNN
 F 2 "Pin_Headers:Pin_Header_Straight_1x02" H 4000 2100 50  0001 C CNN
 F 3 "" H 4000 2100 50  0000 C CNN
@@
 P 3050 2100
 F 0 "P2" H 3050 2250 50  0000 C CNN
-F 1 "Force OFF (NC)" V 3150 2250 50  0000 C CNN
+F 1 "Force off (NC)" V 3150 2250 50  0000 C CNN
 F 2 "Pin_Headers:Pin_Header_Straight_1x02" H 3050 2100 50  0001 C CNN
 F 3 "" H 3050 2100 50  0000 C CNN
@@
 Sense-On
 Text HLabel 3600 1900 1    60   Output ~ 0
-Sense-Powered
+Sense-Sustained
 Wire Notes Line
 	3650 3950 3650 4100
@@
 Connection ~ 3800 3200
 Connection ~ 3900 3200
+Text Notes 3100 1900 1    60   ~ 0
+with RPi\nswitched Relay
+Text Notes 4050 1900 1    60   ~ 0
+with RPi\nswitched Relay
+Text Notes 2050 3850 0    60   ~ 0
+[1, 2]: E-Stop; NC\n[2, 3]: Off; NC  (NB: 2 is shared)\n[4, 5]: On; NO\n
 $EndSCHEMATC

Commit message: Upgrade to new eeschema lib.
Parts:
- P1, P2, P5: symbol CONN_01X02 -> switch-connector-rescue:CONN_01X02-RESCUE-switch-connector
- P3: symbol CONN_01X04 -> switch-connector-rescue:CONN_01X04-RESCUE-switch-connector
- P4: symbol CONN_01X05 -> switch-connector-rescue:CONN_01X05-RESCUE-switch-connector
- P6: symbol CONN_01X03 -> switch-connector-rescue:CONN_01X03-RESCUE-switch-connector
- SW1, SW2, SW3: symbol SW_PUSH -> switch-connector-rescue:SW_PUSH-RESCUE-switch-connector
Connections:
- wire segments 37 -> 51
Changed lines of the file:
@@
-EESchema Schematic File Version 2
-LIBS:power
-LIBS:device
-LIBS:transistors
-LIBS:conn
-LIBS:linear
-LIBS:regul
-LIBS:74xx
-LIBS:cmos4000
-LIBS:adc-dac
-LIBS:memory
-LIBS:xilinx
-LIBS:microcontrollers
-LIBS:dsp
-LIBS:microchip
-LIBS:analog_switches
-LIBS:motorola
-LIBS:texas
-LIBS:intel
-LIBS:audio
-LIBS:interface
-LIBS:digital-audio
-LIBS:philips
-LIBS:display
-LIBS:cypress
-LIBS:siliconi
-LIBS:opto
-LIBS:atmel
-LIBS:contrib
-LIBS:valves
-LIBS:relays
-LIBS:parts
-LIBS:switches
+EESchema Schematic File Version 4
 LIBS:switch-connector-cache
-EELAYER 25 0
+EELAYER 26 0
 EELAYER END
 $Descr A4 11693 8268
@@
 $EndDescr
 $Comp
-L SW_PUSH SW1
+L switch-connector-rescue:SW_PUSH-RESCUE-switch-connector SW1
 U 1 1 57D0AB9F
 P 2650 2600
@@
 $EndComp
 $Comp
-L CONN_01X02 P1
+L switch-connector-rescue:CONN_01X02-RESCUE-switch-connector P1
 U 1 1 57D0AC23
 P 1150 2750
+AR Path="/57D0AC23" Ref="P1"  Part="1"
+AR Path="/58AB5D07/57D0AC23" Ref="P1"  Part="1"
 F 0 "P1" H 1150 2900 50  0000 C CNN
 F 1 "12V" V 1250 2750 50  0000 C CNN
@@
 $EndComp
 $Comp
-L SW_PUSH SW2
+L switch-connector-rescue:SW_PUSH-RESCUE-switch-connector SW2
 U 1 1 57D0AC74
 P 3650 2600
@@
 $EndComp
 $Comp
-L CONN_01X02 P5
+L switch-connector-rescue:CONN_01X02-RESCUE-switch-connector P5
 U 1 1 57D0B52B
 P 4000 2100
+AR Path="/57D0B52B" Ref="P5"  Part="1"
+AR Path="/58AB5D07/57D0B52B" Ref="P5"  Part="1"
 F 0 "P5" H 4000 2250 50  0000 C CNN
 F 1 "Enable on (NO)" V 4100 2100 50  0000 C CNN
@@
 $EndComp
 $Comp
-L CONN_01X02 P2
+L switch-connector-rescue:CONN_01X02-RESCUE-switch-connector P2
 U 1 1 57D0B59A
 P 3050 2100
+AR Path="/57D0B59A" Ref="P2"  Part="1"
+AR Path="/58AB5D07/57D0B59A" Ref="P2"  Part="1"
 F 0 "P2" H 3050 2250 50  0000 C CNN
 F 1 "Force off (NC)" V 3150 2250 50  0000 C CNN
@@
 $EndComp
 $Comp
-L SW_PUSH SW3
+L switch-connector-rescue:SW_PUSH-RESCUE-switch-connector SW3
 U 1 1 57D0C011
 P 1850 2600
@@
 $EndComp
 $Comp
-L CONN_01X04 P3
+L switch-connector-rescue:CONN_01X04-RESCUE-switch-connector P3
 U 1 1 57D0C0C3
 P 3450 2100
@@
 Sustain
 $Comp
-L GND #PWR01
+L power:GND #PWR01
 U 1 1 58AB6D12
 P 1450 3000
@@
 CoilGnd
 $Comp
-L +12V #PWR02
+L power:+12V #PWR02
 U 1 1 58AB7391
 P 1450 2600
@@
 	3900 4300 3900 4250
 Wire Wire Line
-	1350 3000 3700 3000
-Wire Wire Line
-	3800 2850 3800 3450
+	1350 3000 1450 3000
+Wire Wire Line
+	3800 2850 3800 3200
 Wire Wire Line
 	4050 2950 3900 2950
 Wire Wire Line
-	3900 2950 3900 3450
+	3900 2950 3900 3200
 Wire Notes Line
 	3800 3950 3800 4100
@@
 	3950 4300 3950 3950
 Wire Wire Line
-	3100 2600 3350 2600
+	3100 2600 3250 2600
 Connection ~ 3250 2600
 Wire Wire Line
-	3950 2300 3950 2900
+	3950 2300 3950 2400
 Wire Wire Line
 	4050 2300 4050 2950
@@
 Connection ~ 4050 2300
 Wire Wire Line
-	3500 1900 3500 2400
+	3500 1900 3500 2300
 Wire Wire Line
 	3500 2400 3950 2400
 Connection ~ 3950 2400
 Wire Wire Line
-	2150 2600 2350 2600
+	2150 2600 2300 2600
 Wire Wire Line
 	3300 2300 2300 2300
 Wire Wire Line
-	2300 2300 2300 2750
+	2300 2300 2300 2600
 Connection ~ 2300 2600
 Wire Wire Line
-	1350 2600 1550 2600
+	1350 2600 1450 2600
 Wire Wire Line
 	1350 2600 1350 2700
@@
 	3300 2300 3300 1900
 Wire Wire Line
-	3400 1900 3400 2400
+	3400 1900 3400 2300
 Connection ~ 3400 2300
 Connection ~ 3300 2300
@@
 	3600 2300 3600 1900
 $Comp
-L CONN_01X05 P4
+L switch-connector-rescue:CONN_01X05-RESCUE-switch-connector P4
 U 1 1 58AB6DAC
 P 2350 3400
@@
 	2450 3200 2450 2850
 Wire Wire Line
-	2450 2850 3800 2850
-Wire Wire Line
-	3250 2400 3250 2850
+	2450 2850 3250 2850
+Wire Wire Line
+	3250 2400 3250 2600
 Connection ~ 3250 2850
 Wire Wire Line
@@
 Connection ~ 3950 2600
 $Comp
-L CONN_01X03 P6
+L switch-connector-rescue:CONN_01X03-RESCUE-switch-connector P6
 U 1 1 58AB7BE4
 P 3800 3400
@@
 $EndComp
 Wire Wire Line
-	3700 3000 3700 3450
+	3700 3000 3700 3200
 Connection ~ 3700 3200
 Connection ~ 3800 3200
@@
 Text Notes 2050 3850 0    60   ~ 0
 [1, 2]: E-Stop; NC\n[2, 3]: Off; NC  (NB: 2 is shared)\n[4, 5]: On; NO\n
+Wire Wire Line
+	3250 2600 3350 2600
+Wire Wire Line
+	3250 2600 3250 2850
+Wire Wire Line
+	3950 2400 3950 2600
+Wire Wire Line
+	2300 2600 2350 2600
+Wire Wire Line
+	2300 2600 2300 2750
+Wire Wire Line
+	1450 3000 3700 3000
+Wire Wire Line
+	1450 2600 1550 2600
+Wire Wire Line
+	3500 2300 3500 2400
+Wire Wire Line
+	3400 2300 3400 2400
+Wire Wire Line
+	3250 2850 3800 2850
+Wire Wire Line
+	3950 2600 3950 2900
+Wire Wire Line
+	3700 3200 3700 3450
+Wire Wire Line
+	3800 3200 3800 3450
+Wire Wire Line
+	3900 3200 3900 3450
 $EndSCHEMATC

Commit message: A little more silkscreen to ease assembly.
Also:
o enough space for actual connectors for switches and sense outputs
o have inputs for every single switch ('eStop' and 'off' were sharing one)
Parts:
- P3: value Sensing -> 12V Sensing; footprint Pin_Headers:Pin_Header_Straight_1x04 -> Connectors_Molex:Molex_KK-6410-04_04x2.54mm_Straight
- P4: value SwitchConnector -> Switches; footprint Pin_Headers:Pin_Header_Straight_1x05 -> Connectors_Molex:Molex_KK-6410-06_06x2.54mm_Straight; symbol switch-connector-rescue:CONN_01X05-RESCUE-switch-connector -> Connector:Conn_01x06
- P6: value HV-RelayConnector -> HV-Relay
Other:
- note added: "[1, 2]: E-Stop; NC\n[3, 4]: Off; NC (NB: 2 is shared)\n[5, 6]: On; NO\n"
- note removed: "[1, 2]: E-Stop; NC\n[2, 3]: Off; NC (NB: 2 is shared)\n[4, 5]: On; NO\n"
Changed lines of the file:
@@
 P 3450 2100
 F 0 "P3" H 3450 2350 50  0000 C CNN
-F 1 "Sensing" V 3550 2100 50  0000 C CNN
-F 2 "Pin_Headers:Pin_Header_Straight_1x04" H 3450 2100 50  0001 C CNN
+F 1 "12V Sensing" V 3550 2100 50  0000 C CNN
+F 2 "Connectors_Molex:Molex_KK-6410-04_04x2.54mm_Straight" H 3450 2100 50  0001 C CNN
 F 3 "" H 3450 2100 50  0000 C CNN
 	1    3450 2100
@@
 Connection ~ 3950 2400
 Wire Wire Line
-	2150 2600 2300 2600
+	2150 2600 2250 2600
 Wire Wire Line
 	3300 2300 2300 2300
@@
 	3600 2300 3600 1900
 $Comp
-L switch-connector-rescue:CONN_01X05-RESCUE-switch-connector P4
+L Connector:Conn_01x06 P4
 U 1 1 58AB6DAC
 P 2350 3400
 F 0 "P4" V 2222 3678 50  0000 L CNN
-F 1 "SwitchConnector" V 2450 3100 50  0000 L CNN
-F 2 "Pin_Headers:Pin_Header_Straight_1x05" H 2350 3400 50  0001 C CNN
+F 1 "Switches" V 2450 3100 50  0000 L CNN
+F 2 "Connectors_Molex:Molex_KK-6410-06_06x2.54mm_Straight" H 2350 3400 50  0001 C CNN
 F 3 "" H 2350 3400 50  0000 C CNN
 	1    2350 3400
@@
 Connection ~ 1550 2600
 Wire Wire Line
-	2300 2750 2250 2750
-Wire Wire Line
-	2250 2750 2250 3200
-Wire Wire Line
 	2950 2600 2950 2800
 Wire Wire Line
-	2950 2800 2350 2800
-Wire Wire Line
-	2350 2800 2350 3200
+	2950 2800 2450 2800
 Connection ~ 2950 2600
-Wire Wire Line
-	2450 3200 2450 2850
-Wire Wire Line
-	2450 2850 3250 2850
 Wire Wire Line
 	3250 2400 3250 2600
 Connection ~ 3250 2850
-Wire Wire Line
-	2550 3200 2550 2900
-Wire Wire Line
-	2550 2900 3950 2900
 Connection ~ 3950 2600
 $Comp
@@
 P 3800 3400
 F 0 "P6" V 3672 3212 50  0000 R CNN
-F 1 "HV-RelayConnector" V 3763 3212 50  0000 R CNN
+F 1 "HV-Relay" V 3763 3212 50  0000 R CNN
 F 2 "Pin_Headers:Pin_Header_Straight_1x04" H 3809 3212 50  0001 R CNN
 F 3 "" H 3800 3400 50  0000 C CNN
@@
 with RPi\nswitched Relay
 Text Notes 2050 3850 0    60   ~ 0
-[1, 2]: E-Stop; NC\n[2, 3]: Off; NC  (NB: 2 is shared)\n[4, 5]: On; NO\n
+[1, 2]: E-Stop; NC\n[3, 4]: Off; NC  (NB: 2 is shared)\n[5, 6]: On; NO\n
 Wire Wire Line
 	3250 2600 3350 2600
@@
 	2300 2600 2350 2600
 Wire Wire Line
-	2300 2600 2300 2750
-Wire Wire Line
 	1450 3000 3700 3000
 Wire Wire Line
@@
 Wire Wire Line
 	3900 3200 3900 3450
+Wire Wire Line
+	2650 3200 2650 2900
+Wire Wire Line
+	2650 2900 3950 2900
+Wire Wire Line
+	2550 3200 2550 2850
+Wire Wire Line
+	2550 2850 3250 2850
+Wire Wire Line
+	2450 3200 2450 2800
+Wire Wire Line
+	2250 2600 2250 3200
+Connection ~ 2250 2600
+Wire Wire Line
+	2250 2600 2300 2600
+Wire Wire Line
+	2350 2600 2350 3200
+Connection ~ 2350 2600
 $EndSCHEMATC

Commit message: Add screw terminal for 12V
Parts:
- P1: footprint Pin_Headers:Pin_Header_Straight_1x02 -> TerminalBlock_RND:TerminalBlock_RND_205-00045_Pitch5.00mm; symbol switch-connector-rescue:CONN_01X02-RESCUE-switch-connector -> Connector:Conn_01x02
- P6: footprint Pin_Headers:Pin_Header_Straight_1x04 -> TerminalBlock_RND:TerminalBlock_RND_205-00047_Pitch5.00mm; symbol switch-connector-rescue:CONN_01X03-RESCUE-switch-connector -> Connector:Conn_01x03
Changed lines of the file:
@@
 $EndComp
 $Comp
-L switch-connector-rescue:CONN_01X02-RESCUE-switch-connector P1
+L Connector:Conn_01x02 P1
 U 1 1 57D0AC23
-P 1150 2750
+P 1150 2800
 AR Path="/57D0AC23" Ref="P1"  Part="1"
 AR Path="/58AB5D07/57D0AC23" Ref="P1"  Part="1"
-F 0 "P1" H 1150 2900 50  0000 C CNN
-F 1 "12V" V 1250 2750 50  0000 C CNN
-F 2 "Pin_Headers:Pin_Header_Straight_1x02" H 1150 2750 50  0001 C CNN
-F 3 "" H 1150 2750 50  0000 C CNN
-	1    1150 2750
+F 0 "P1" H 1150 2950 50  0000 C CNN
+F 1 "12V" H 1150 2600 50  0000 C CNN
+F 2 "TerminalBlock_RND:TerminalBlock_RND_205-00045_Pitch5.00mm" H 1150 2800 50  0001 C CNN
+F 3 "" H 1150 2800 50  0000 C CNN
+	1    1150 2800
 	-1   0    0    1
 $EndComp
@@
 Connection ~ 3950 2600
 $Comp
-L switch-connector-rescue:CONN_01X03-RESCUE-switch-connector P6
+L Connector:Conn_01x03 P6
 U 1 1 58AB7BE4
 P 3800 3400
 F 0 "P6" V 3672 3212 50  0000 R CNN
 F 1 "HV-Relay" V 3763 3212 50  0000 R CNN
-F 2 "Pin_Headers:Pin_Header_Straight_1x04" H 3809 3212 50  0001 R CNN
+F 2 "TerminalBlock_RND:TerminalBlock_RND_205-00047_Pitch5.00mm" H 3809 3212 50  0001 R CNN
 F 3 "" H 3800 3400 50  0000 C CNN
 	1    3800 3400

Commit message: Update schematic to refined design.
(PCB still needs to be adapted)
Parts:
- removed P2: Force off (NC), Pin_Headers:Pin_Header_Straight_1x02, symbol switch-connector-rescue:CONN_01X02-RESCUE-switch-connector
- removed P3: 12V Sensing, Connectors_Molex:Molex_KK-6410-04_04x2.54mm_Straight, symbol switch-connector-rescue:CONN_01X04-RESCUE-switch-connector
- removed P5: Enable on (NO), Pin_Headers:Pin_Header_Straight_1x02, symbol switch-connector-rescue:CONN_01X02-RESCUE-switch-connector
- removed SW1: NC: Off, symbol switch-connector-rescue:SW_PUSH-RESCUE-switch-connector
- removed SW2: NO: On, symbol switch-connector-rescue:SW_PUSH-RESCUE-switch-connector
- removed SW3: NC: E-Stop, symbol switch-connector-rescue:SW_PUSH-RESCUE-switch-connector
- added C1: 100u, Capacitors_THT:CP_Radial_D8.0mm_P3.50mm, symbol device:CP
- added P3: Pi, symbol Connector:Conn_02x05_Odd_Even
- added P4: 5V, Pin_Headers:Pin_Header_Straight_1x02_Pitch2.54mm, symbol Connector:Conn_01x02
- added P5: RL-In, Pin_Headers:Pin_Header_Straight_1x02_Pitch2.54mm, symbol Connector:Conn_01x02
- added P6: UART, Pin_Headers:Pin_Header_Straight_1x02_Pitch2.54mm, symbol Connector:Conn_01x02
- added R1, R2: 1k, Resistors_THT:R_Axial_DIN0411_L9.9mm_D3.6mm_P12.70mm_Horizontal, symbol device:R
- added RL2: Trigger off (NC), Pin_Headers:Pin_Header_Straight_1x02_Pitch2.54mm, symbol Switch:SW_Push_Open
- added RL3: Enable On (NO), Pin_Headers:Pin_Header_Straight_1x02_Pitch2.54mm, symbol Switch:SW_Push
- P2: renamed from P4; footprint Connectors_Molex:Molex_KK-6410-06_06x2.54mm_Straight -> Connectors_JST:JST_XH_B06B-XH-A_06x2.50mm_Straight
- renumbered P6 to Conn-RL1
Connections:
- net labels added: +5V, Off-B, On-B, RL-Trigger-Off, RL-Trigger-On, RX, Sense-EStop, SenseRelay, TX
- net labels removed: Sense-E-Stop, Sense-Off, Sense-On, Sense-Sustained
- wire segments 51 -> 52
Other:
- note added: "Relay Voltage"
- note added: "Switches from Trigger Relays"
- note added: "[1, 2]: E-Stop; NC\n[3, 4]: Off; NC \n[5, 6]: On; NO\n"
- note removed: "[1, 2]: E-Stop; NC\n[3, 4]: Off; NC (NB: 2 is shared)\n[5, 6]: On; NO\n"
- note removed: "with RPi\nswitched Relay"
