File: hardware/switch-connector/switch-connector.kicad_pcb (KiCad board)
At the start: 2 copper layers, 38 x 28 mm, 12 parts, among them J1 Relay Control, J2 RFID connect, P1 12V, P2 Switches, P3 Pi

Commit message: Update Schematic image in README; smallish tweaks in PCB.
Routing:
- net GND: track 60.8 -> 63.0 mm
- added copper zone on F.Cu, net GND
Other:
- board text added: "<- 20mm ->"
- board text added: "<- 30mm (M3) ->"
- board text added: "github.com/noisebridge/sparkle-switch"
- board text removed: "Trg. Relay"
Changed lines of the file:
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@@
   (general
     (thickness 1.6)
-    (drawings 75)
-    (tracks 87)
+    (drawings 76)
+    (tracks 88)
     (zones 0)
     (modules 12)
@@
     (user_trace_width 2)
     (trace_clearance 0.4)
-    (zone_clearance 0.8)
+    (zone_clearance 0.6)
     (zone_45_only no)
     (trace_min 0.2)
@@
     (descr "JST PH series connector, B4B-PH-K, top entry type, through hole, Datasheet: http://www.jst-mfg.com/product/pdf/eng/ePH.pdf")
     (tags "connector jst ph")
-    (fp_text reference J1 (at 9.017 4.826 90) (layer F.SilkS)
+    (fp_text reference J1 (at 8.89 4.445 180) (layer F.SilkS)
       (effects (font (size 1 1) (thickness 0.15)))
     )
@@
     (pad 1 np_thru_hole circle (at 0 0) (size 3.2 3.2) (drill 3.2) (layers *.Cu *.Mask F.SilkS))
   )
+  (gr_text "<- 20mm ->" (at 191.206 111.97 90) (layer B.SilkS)
+    (effects (font (size 1 1) (thickness 0.2)) (justify mirror))
+  )
+  (gr_text "<- 30mm (M3) ->" (at 178.633 124.162) (layer B.SilkS)
+    (effects (font (size 1 1) (thickness 0.2)) (justify mirror))
+  )
+  (gr_text github.com/noisebridge/sparkle-switch (at 176.982 118.066) (layer B.SilkS)
+    (effects (font (size 1.2 1.2) (thickness 0.2)) (justify mirror))
+  )
   (gr_line (start 167.767 114.129) (end 167.767 113.875) (layer B.SilkS) (width 0.2))
   (gr_text "Mains Relay" (at 162.25 117.939) (layer F.SilkS)
@@
     (effects (font (size 1 1) (thickness 0.15)))
   )
-  (gr_text "Trg. Relay" (at 176.474 132.036) (layer F.SilkS)
-    (effects (font (size 0.7 0.7) (thickness 0.12)))
-  )
-  (gr_text "Trg. Relay" (at 162.25 95.587) (layer F.SilkS)
-    (effects (font (size 0.7 0.7) (thickness 0.12)))
-  )
   (gr_text "\"OFF\" (NC)" (at 165.298 121.622 90) (layer F.SilkS)
     (effects (font (size 0.7 0.7) (thickness 0.12)))
@@
     (effects (font (size 0.7 0.7) (thickness 0.12)))
   )
-  (gr_text "H.Zeller 2018" (at 183.078 98.762) (layer F.SilkS)
-    (effects (font (size 1 1) (thickness 0.15)))
+  (gr_text "H.Zeller 2018" (at 178.76 107.271) (layer B.SilkS)
+    (effects (font (size 1 1) (thickness 0.15)) (justify mirror))
   )
   (gr_text "Mains Relay" (at 162.123 105.747) (layer F.SilkS)
     (effects (font (size 0.8 0.8) (thickness 0.12)))
   )
-  (gr_text "Trg. Relay" (at 188.92 101.81 90) (layer F.SilkS)
+  (gr_text "Trigger Relays" (at 183.332 98.635) (layer F.SilkS)
     (effects (font (size 1 1) (thickness 0.15)))
   )
@@
   (segment (start 171.521 99.872) (end 171.96401 99.42899) (width 1.5) (layer B.Cu) (net 1))
   (segment (start 171.521 102.572) (end 171.521 99.872) (width 1.5) (layer B.Cu) (net 1))
-  (segment (start 171.521 105.120647) (end 171.521 102.572) (width 1.5) (layer F.Cu) (net 1))
-  (segment (start 168.736979 107.904667) (end 171.521 105.120647) (width 1.5) (layer F.Cu) (net 1))
   (segment (start 162.123 115.399) (end 162.170849 115.399) (width 1.5) (layer F.Cu) (net 1))
-  (segment (start 168.736979 108.83287) (end 168.736979 107.904667) (width 1.5) (layer F.Cu) (net 1))
-  (segment (start 162.170849 115.399) (end 168.736979 108.83287) (width 1.5) (layer F.Cu) (net 1))
   (segment (start 192.310853 115.787) (end 193.619 115.787) (width 1.5) (layer B.Cu) (net 1))
   (segment (start 184.80387 115.787) (end 192.310853 115.787) (width 1.5) (layer B.Cu) (net 1))
   (segment (start 182.697 113.68013) (end 184.80387 115.787) (width 1.5) (layer B.Cu) (net 1))
   (segment (start 182.697 113.24) (end 182.697 113.68013) (width 1.5) (layer B.Cu) (net 1))
+  (segment (start 166.830648 114.374352) (end 165.806 115.399) (width 1.5) (layer F.Cu) (net 1))
+  (segment (start 166.830648 109.811) (end 166.830648 114.374352) (width 1.5) (layer F.Cu) (net 1))
+  (segment (start 171.521 102.572) (end 171.521 105.120648) (width 1.5) (layer F.Cu) (net 1))
+  (segment (start 165.806 115.399) (end 162.123 115.399) (width 1.5) (layer F.Cu) (net 1))
+  (segment (start 171.521 105.120648) (end 166.830648 109.811) (width 1.5) (layer F.Cu) (net 1))
   (segment (start 174.191999 123.647001) (end 176.876435 123.647001) (width 1.5) (layer F.Cu) (net 2))
   (segment (start 172.664 122.119002) (end 174.191999 123.647001) (width 1.5) (layer F.Cu) (net 2))
@@
   (segment (start 180.157 114.314294) (end 185.164 119.321294) (width 1.5) (layer B.Cu) (net 12))
   (zone (net 1) (net_name GND) (layer B.Cu) (hatch edge 0.508)
-    (connect_pads (clearance 0.8))
+    (connect_pads (clearance 0.6))
     (min_thickness 0.254)
     (fill yes (arc_segments 16) (thermal_gap 0.508) (thermal_bridge_width 0.508))
     (polygon
       (pts
-        (xy 158.75 97.79) (xy 197.485 97.79) (xy 197.485 125.73) (xy 158.75 125.73)
+        (xy 157.805 97.79) (xy 196.54 97.79) (xy 196.54 125.73) (xy 157.805 125.73)
       )
     )
+  )
+  (zone (net 1) (net_name GND) (layer F.Cu) (hatch edge 0.508)
+    (connect_pads (clearance 0.6))
+    (min_thickness 0.254)
+    (fill yes (arc_segments 16) (thermal_gap 0.508) (thermal_bridge_width 0.508))
+    (polygon
+      (pts
+        (xy 157.678 97.917) (xy 196.413 97.917) (xy 196.413 125.857) (xy 157.678 125.857)
+      )
+    )
